Commit message: Updated model for gazebo
Still not entirely working

File: src/tfr_description/xacro/model.xacro (robot description, xacro)
@@ -5,3 +5,9 @@
   <xacro:include filename="model_base.xacro"/>
   <xacro:include filename="model_arm.xacro"/>
+  <gazebo>
+    <plugin name="gazebo_ros_control" filename="libgazebo_ros_control.so">
+      <robotNamespace>/</robotNamespace>
+      <robotSimType>gazebo_ros_control/DefaultRobotHWSim</robotSimType>
+    </plugin>
+  </gazebo>
 </robot>

File: src/tfr_description/xacro/model_arm.xacro (robot description, xacro)
@@ -15,4 +15,9 @@
       <origin xyz="0 0 ${turntable_height/2}" rpy="0 0 ${pi}" />
     </collision>
+    <!-- test -->
+    <inertial>
+      <mass value="1.0" />
+      <inertia ixx="1.0" ixy="0.0" ixz="0.0" iyy="1.0" iyz="0.0" izz="1.0"/>
+    </inertial>
   </link>
   <joint name="turntable_joint" type="revolute">
@@ -49,4 +54,9 @@
       <origin xyz="${-lower_arm_height/2} 0 ${14*itom}" />
     </collision>
+    <!-- test -->
+    <inertial>
+      <mass value="1.0" />
+      <inertia ixx="1.0" ixy="0.0" ixz="0.0" iyy="1.0" iyz="0.0" izz="1.0"/>
+    </inertial>
   </link>
   <joint name="lower_arm_joint" type="revolute">
@@ -82,4 +92,9 @@
       </geometry>
     </collision>
+    <!-- test -->
+    <inertial>
+      <mass value="1.0" />
+      <inertia ixx="1.0" ixy="0.0" ixz="0.0" iyy="1.0" iyz="0.0" izz="1.0"/>
+    </inertial>
   </link>
   <joint name="lower_arm_bottom_joint" type="fixed">
@@ -101,4 +116,9 @@
       <origin xyz="${0.125*itom} 0 ${-(lower_arm_length - lower_arm_primary_length) / 2 * sqrt2}" rpy="0 0 0" />
     </collision>
+    <!-- test -->
+    <inertial>
+      <mass value="1.0" />
+      <inertia ixx="1.0" ixy="0.0" ixz="0.0" iyy="1.0" iyz="0.0" izz="1.0"/>
+    </inertial>
   </link>
   <joint name="lower_arm_slope_joint" type="fixed">
@@ -120,4 +140,9 @@
       <origin xyz="${-upper_arm_height/2} 0 ${upper_arm_length/2}" />
     </collision>
+    <!-- test -->
+    <inertial>
+      <mass value="1.0" />
+      <inertia ixx="1.0" ixy="0.0" ixz="0.0" iyy="1.0" iyz="0.0" izz="1.0"/>
+    </inertial>
   </link>
   <joint name="upper_arm_joint" type="revolute">
@@ -155,4 +180,9 @@
       <origin xyz="${scoop_length/2} 0 ${scoop_diameter/4}" />
     </collision>
+    <!-- test -->
+    <inertial>
+      <mass value="1.0" />
+      <inertia ixx="1.0" ixy="0.0" ixz="0.0" iyy="1.0" iyz="0.0" izz="1.0"/>
+    </inertial>
   </link>
   <joint name="scoop_joint" type="revolute">

Commit message: Model of arm works

File: src/tfr_description/xacro/model.xacro (robot description, xacro)
@@ -3,5 +3,11 @@
   <!-- Top-level robot description -->
   <xacro:include filename="model_constants.xacro"/>
-  <xacro:include filename="model_base.xacro"/>
+  <!-- <xacro:include filename="model_base.xacro"/> -->
   <xacro:include filename="model_arm.xacro"/>
+  <gazebo>
+    <plugin name="gazebo_ros_control" filename="libgazebo_ros_control.so">
+      <robotNamespace>/</robotNamespace>
+      <!-- <robotSimType>gazebo_ros_control/DefaultRobotHWSim</robotSimType> -->
+    </plugin>
+  </gazebo>
 </robot>

File: src/tfr_description/xacro/model_arm.xacro (robot description, xacro)
@@ -1,4 +1,15 @@
 <?xml version="1.0"?>
 <robot xmlns:xacro="http://www.ros.org/wiki/xacro" name="excavator">
+  <!-- attatch robot to world frame-->
+  <link name="world">
+    <inertial>
+      <mass value="${100.0}" />
+      <inertia ixx="100.0" ixy="0.0" ixz="0.0" iyy="100.0" iyz="0.0" izz="100.0"/>
+    </inertial>
+  </link>
+  <joint name="fixed" type="fixed">
+    <parent link="world"/>
+    <child link="turntable"/>
+  </joint>
   <!--DIGGING ARM-->
   <link name="turntable">
@@ -15,6 +26,15 @@
       <origin xyz="0 0 ${turntable_height/2}" rpy="0 0 ${pi}" />
     </collision>
-  </link>
-  <joint name="turntable_joint" type="revolute">
+    <!-- test -->
+    <inertial>
+      <mass value="20.0" />
+      <!--<inertia ixx="${0.0833333 * turntable_mass * (3.0 * turntable_radius * turntable_radius + turntable_height * turntable_height)}" ixy="0.0" ixz="0.0"
+        iyy="${0.0833333 * turntable_mass * (3.0 * turntable_radius * turntable_radius + turntable_height * turntable_height)}" iyz="0.0"
+        izz="${0.5 * turntable_mass * turntable_radius * turntable_radius}" />-->
+      <inertia ixx="20.0" ixy="0.0" ixz="0.0" iyy="20.0" iyz="0.0" izz="20.0"/>
+    </inertial>
+  </link>
+  <!--Removed joint because for my simulation I am not including the base-->
+  <!--<joint name="turntable_joint" type="revolute">
     <parent link="base_link" />
     <child link="turntable" />
@@ -25,5 +45,5 @@
   <transmission name="turntable_tran">
     <type>transmission_interface/SimpleTransmission</type>
-    <joint name="turn_to_base">
+    <joint name="turntable_joint">
       <hardwareInterface>hardware_interface/EffortJointInterface
       </hardwareInterface>
@@ -35,5 +55,5 @@
       <motorTorqueConstant>1</motorTorqueConstant>
     </actuator>
-  </transmission>
+  </transmission>-->
   <link name="lower_arm">
     <visual>
@@ -49,4 +69,12 @@
       <origin xyz="${-lower_arm_height/2} 0 ${14*itom}" />
     </collision>
+    <!-- test -->
+    <inertial>
+      <mass value="15.0" />
+      <!--<inertia ixx="${0.0833333 * lower_arm_mass * (lower_arm_width*lower_arm_width + lower_arm_primary_length*lower_arm_primary_length)}" ixy="0.0" ixz="0.0"
+        iyy="${0.0833333 * lower_arm_mass * (lower_arm_height*lower_arm_height + lower_arm_primary_length*lower_arm_primary_length)}" iyz="0.0"
+        izz="${0.0833333 * lower_arm_mass * (lower_arm_height*lower_arm_height + lower_arm_width*lower_arm_width)}" />-->
+      <inertia ixx="15.0" ixy="0.0" ixz="0.0" iyy="15.0" iyz="0.0" izz="15.0"/>
+    </inertial>
   </link>
   <joint name="lower_arm_joint" type="revolute">
@@ -60,5 +88,5 @@
   <transmission name="lower_arm_tran">
     <type>transmission_interface/SimpleTransmission</type>
-    <joint name="lower_to_turn">
+    <joint name="lower_arm_joint">
       <hardwareInterface>hardware_interface/EffortJointInterface
       </hardwareInterface>
@@ -82,4 +110,10 @@
       </geometry>
     </collision>
+    <!-- test -->
+    <inertial>
+      <mass value="15.0" />
+      <!--<inertia ixx="0.0833333 * lower_arm_mass" ixy="0.0" ixz="0.0" iyy="0.0833333 * lower_arm_mass" iyz="0.0" izz="0.0833333 * lower_arm_mass"/> -->
+      <inertia ixx="15.0" ixy="0.0" ixz="0.0" iyy="15.0" iyz="0.0" izz="15.0"/>
+    </inertial>
   </link>
   <joint name="lower_arm_bottom_joint" type="fixed">
@@ -101,4 +135,10 @@
       <origin xyz="${0.125*itom} 0 ${-(lower_arm_length - lower_arm_primary_length) / 2 * sqrt2}" rpy="0 0 0" />
     </collision>
+    <!-- test -->
+    <inertial>
+      <mass value="15.0" />
+      <!--<inertia ixx="0.0833333 * lower_arm_mass" ixy="0.0" ixz="0.0" iyy="0.0833333 * lower_arm_mass" iyz="0.0" izz="0.0833333 * lower_arm_mass"/>  -->
+      <inertia ixx="15.0" ixy="0.0" ixz="0.0" iyy="15.0" iyz="0.0" izz="15.0"/>
+    </inertial>
   </link>
   <joint name="lower_arm_slope_joint" type="fixed">
@@ -120,4 +160,12 @@
       <origin xyz="${-upper_arm_height/2} 0 ${upper_arm_length/2}" />
     </collision>
+    <!-- test -->
+    <inertial>
+      <mass value="10.0" />
+      <!--<inertia ixx="${0.0833333 * upper_arm_mass * (upper_arm_width*upper_arm_width + upper_arm_length*upper_arm_length)}" ixy="0.0" ixz="0.0"
+        iyy="${0.0833333 * upper_arm_mass * (upper_arm_height*upper_arm_height + upper_arm_length*upper_arm_length)}" iyz="0.0"
+        izz="${0.0833333 * upper_arm_mass * (upper_arm_height*upper_arm_height + upper_arm_width*upper_arm_width)}" /> -->
+      <inertia ixx="10.0" ixy="0.0" ixz="0.0" iyy="10.0" iyz="0.0" izz="10.0"/>
+    </inertial>
   </link>
   <joint name="upper_arm_joint" type="revolute">
@@ -131,5 +179,5 @@
   <transmission name="upper_arm_tran">
     <type>transmission_interface/SimpleTransmission</type>
-    <joint name="upper_to_lower">
+    <joint name="upper_arm_joint">
       <hardwareInterface>hardware_interface/EffortJointInterface
       </hardwareInterface>
@@ -155,4 +203,12 @@
       <origin xyz="${scoop_length/2} 0 ${scoop_diameter/4}" />
     </collision>
+    <!-- test -->
+    <inertial>
+      <mass value="5.0" />
+      <!--<inertia ixx="${0.0833333 * scoop_mass * (scoop_width*scoop_width + (scoop_diameter/2)*(scoop_diameter/2))}" ixy="0.0" ixz="0.0"
+        iyy="${0.0833333 * scoop_mass * (scoop_length*scoop_length + (scoop_diameter/2)*(scoop_diameter/2))}" iyz="0.0"
+        izz="${0.0833333 * scoop_mass * (scoop_length*scoop_length + scoop_width*scoop_width)}" />-->
+      <inertia ixx="5.0" ixy="0.0" ixz="0.0" iyy="5.0" iyz="0.0" izz="5.0"/>
+    </inertial>
   </link>
   <joint name="scoop_joint" type="revolute">
@@ -166,5 +222,5 @@
   <transmission name="scoop_tran">
     <type>transmission_interface/SimpleTransmission</type>
-    <joint name="end_to_arm">
+    <joint name="scoop_joint">
       <hardwareInterface>hardware_interface/EffortJointInterface
       </hardwareInterface>

File: src/tfr_description/xacro/model_constants.xacro (robot description, xacro)
@@ -9,4 +9,5 @@
   <xacro:property name="sqrt2" value="1.41421" />
   <!-- Drivebase parameters -->
+  <xacro:property name="base_mass" value="${25.0}"/>
   <xacro:property name="base_length" value="${50*itom}" />
   <xacro:property name="tube_width" value="${2*itom}" />
@@ -31,4 +32,5 @@
   <xacro:property name="bin_back_offset" value="${6.5*itom}" />
   <!-- Turntable parameters -->
+  <xacro:property name="turntable_mass" value="${25.0}"/>
   <xacro:property name="turntable_radius" value="${4.92*itom}" />
   <!-- 1" in model plus undefined height for mounting and extra components -->
@@ -36,4 +38,5 @@
   <xacro:property name="turntable_height" value="${2.25*itom}" />
   <!-- Lower arm parameters -->
+  <xacro:property name="lower_arm_mass" value="${15.0}"/>
   <xacro:property name="lower_arm_length" value="${22*itom}" />
   <xacro:property name="lower_arm_primary_length" value="${16*itom}" />
@@ -43,4 +46,5 @@
   <xacro:property name="lower_arm_max" value="1.55" />
   <!-- Upper arm parameters -->
+  <xacro:property name="upper_arm_mass" value="${10.0}"/>
   <xacro:property name="upper_arm_length" value="${20*itom}" />
   <xacro:property name="upper_arm_width" value="${4.75*itom}" />
@@ -49,4 +53,5 @@
   <xacro:property name="upper_arm_max" value="2.4"/>
   <!-- Scoop parameters -->
+  <xacro:property name="scoop_mass" value="${5.0}"/>
   <xacro:property name="scoop_width" value="${8.5*itom}" />
   <xacro:property name="scoop_length" value="${12*itom}" />

Commit message: Description changed to model the arm in gazebo

File: src/tfr_description/xacro/model.xacro (robot description, xacro)
@@ -3,9 +3,9 @@
   <!-- Top-level robot description -->
   <xacro:include filename="model_constants.xacro"/>
-  <xacro:include filename="model_base.xacro"/>
+  <!--<xacro:include filename="model_base.xacro"/> -->
   <xacro:include filename="model_arm.xacro"/>
   <gazebo>
     <plugin name="gazebo_ros_control" filename="libgazebo_ros_control.so">
-      <robotNamespace>/</robotNamespace>
+      <robotNamespace>/tfr_arm</robotNamespace>
       <robotSimType>gazebo_ros_control/DefaultRobotHWSim</robotSimType>
     </plugin>

File: src/tfr_description/xacro/model_arm.xacro (robot description, xacro)
@@ -1,4 +1,15 @@
 <?xml version="1.0"?>
 <robot xmlns:xacro="http://www.ros.org/wiki/xacro" name="excavator">
+  <!-- attatch robot to world frame -->
+  <link name="world">
+    <!--<inertial>
+      <mass value="${100.0}" />
+      <inertia ixx="100.0" ixy="0.0" ixz="0.0" iyy="100.0" iyz="0.0" izz="100.0"/>
+    </inertial>-->
+  </link>
+  <joint name="fixed" type="fixed">
+    <parent link="world"/>
+    <child link="turntable"/>
+  </joint>
   <!--DIGGING ARM-->
   <link name="turntable">
@@ -17,9 +28,13 @@
     <!-- test -->
     <inertial>
-      <mass value="1.0" />
-      <inertia ixx="1.0" ixy="0.0" ixz="0.0" iyy="1.0" iyz="0.0" izz="1.0"/>
-    </inertial>
-  </link>
-  <joint name="turntable_joint" type="revolute">
+      <mass value="20.0" />
+      <!--<inertia ixx="${0.0833333 * turntable_mass * (3.0 * turntable_radius * turntable_radius + turntable_height * turntable_height)}" ixy="0.0" ixz="0.0"
+        iyy="${0.0833333 * turntable_mass * (3.0 * turntable_radius * turntable_radius + turntable_height * turntable_height)}" iyz="0.0"
+        izz="${0.5 * turntable_mass * turntable_radius * turntable_radius}" />-->
+      <inertia ixx="20.0" ixy="0.0" ixz="0.0" iyy="20.0" iyz="0.0" izz="20.0"/>
+    </inertial>
+  </link>
+  <!--Removed joint because for my simulation I am not including the base-->
+  <!--<joint name="turntable_joint" type="revolute">
     <parent link="base_link" />
     <child link="turntable" />
@@ -30,5 +45,5 @@
   <transmission name="turntable_tran">
     <type>transmission_interface/SimpleTransmission</type>
-    <joint name="turn_to_base">
+    <joint name="turntable_joint">
       <hardwareInterface>hardware_interface/EffortJointInterface
       </hardwareInterface>
@@ -40,5 +55,5 @@
       <motorTorqueConstant>1</motorTorqueConstant>
     </actuator>
-  </transmission>
+  </transmission>-->
   <link name="lower_arm">
     <visual>
@@ -56,6 +71,9 @@
     <!-- test -->
     <inertial>
-      <mass value="1.0" />
-      <inertia ixx="1.0" ixy="0.0" ixz="0.0" iyy="1.0" iyz="0.0" izz="1.0"/>
+      <mass value="15.0" />
+      <!--<inertia ixx="${0.0833333 * lower_arm_mass * (lower_arm_width*lower_arm_width + lower_arm_primary_length*lower_arm_primary_length)}" ixy="0.0" ixz="0.0"
+        iyy="${0.0833333 * lower_arm_mass * (lower_arm_height*lower_arm_height + lower_arm_primary_length*lower_arm_primary_length)}" iyz="0.0"
+        izz="${0.0833333 * lower_arm_mass * (lower_arm_height*lower_arm_height + lower_arm_width*lower_arm_width)}" />-->
+      <inertia ixx="15.0" ixy="0.0" ixz="0.0" iyy="15.0" iyz="0.0" izz="15.0"/>
     </inertial>
   </link>
@@ -70,10 +88,14 @@
   <transmission name="lower_arm_tran">
     <type>transmission_interface/SimpleTransmission</type>
-    <joint name="lower_to_turn">
-      <hardwareInterface>hardware_interface/EffortJointInterface
+    <joint name="lower_arm_joint">
+      <!--<hardwareInterface>hardware_interface/EffortJointInterface
+      </hardwareInterface>-->
+      <hardwareInterface>hardware_interface/PositionJointInterface
       </hardwareInterface>
     </joint>
     <actuator name="lower_motor">
-      <hardwareInterface>hardware_interface/EffortJointInterface
+      <!--<hardwareInterface>hardware_interface/EffortJointInterface
+      </hardwareInterface>-->
+      <hardwareInterface>hardware_interface/PositionJointInterface
       </hardwareInterface>
       <mechanicalReduction>1</mechanicalReduction>
@@ -94,6 +116,7 @@
     <!-- test -->
     <inertial>
-      <mass value="1.0" />
-      <inertia ixx="1.0" ixy="0.0" ixz="0.0" iyy="1.0" iyz="0.0" izz="1.0"/>
+      <mass value="15.0" />
+      <!--<inertia ixx="0.0833333 * lower_arm_mass" ixy="0.0" ixz="0.0" iyy="0.0833333 * lower_arm_mass" iyz="0.0" izz="0.0833333 * lower_arm_mass"/> -->
+      <inertia ixx="15.0" ixy="0.0" ixz="0.0" iyy="15.0" iyz="0.0" izz="15.0"/>
     </inertial>
   </link>
@@ -118,6 +141,7 @@
     <!-- test -->
     <inertial>
-      <mass value="1.0" />
-      <inertia ixx="1.0" ixy="0.0" ixz="0.0" iyy="1.0" iyz="0.0" izz="1.0"/>
+      <mass value="15.0" />
+      <!--<inertia ixx="0.0833333 * lower_arm_mass" ixy="0.0" ixz="0.0" iyy="0.0833333 * lower_arm_mass" iyz="0.0" izz="0.0833333 * lower_arm_mass"/>  -->
+      <inertia ixx="15.0" ixy="0.0" ixz="0.0" iyy="15.0" iyz="0.0" izz="15.0"/>
     </inertial>
   </link>
@@ -142,6 +166,9 @@
     <!-- test -->
     <inertial>
-      <mass value="1.0" />
-      <inertia ixx="1.0" ixy="0.0" ixz="0.0" iyy="1.0" iyz="0.0" izz="1.0"/>
+      <mass value="10.0" />
+      <!--<inertia ixx="${0.0833333 * upper_arm_mass * (upper_arm_width*upper_arm_width + upper_arm_length*upper_arm_length)}" ixy="0.0" ixz="0.0"
+        iyy="${0.0833333 * upper_arm_mass * (upper_arm_height*upper_arm_height + upper_arm_length*upper_arm_length)}" iyz="0.0"
+        izz="${0.0833333 * upper_arm_mass * (upper_arm_height*upper_arm_height + upper_arm_width*upper_arm_width)}" /> -->
+      <inertia ixx="10.0" ixy="0.0" ixz="0.0" iyy="10.0" iyz="0.0" izz="10.0"/>
     </inertial>
   </link>
@@ -156,10 +183,10 @@
   <transmission name="upper_arm_tran">
     <type>transmission_interface/SimpleTransmission</type>
-    <joint name="upper_to_lower">
-      <hardwareInterface>hardware_interface/EffortJointInterface
+    <joint name="upper_arm_joint">
+      <hardwareInterface>hardware_interface/PositionJointInterface
       </hardwareInterface>
     </joint>
     <actuator name="upper_motor">
-      <hardwareInterface>hardware_interface/EffortJointInterface
+      <hardwareInterface>hardware_interface/PositionJointInterface
       </hardwareInterface>
       <mechanicalReduction>1</mechanicalReduction>
@@ -182,6 +209,9 @@
     <!-- test -->
     <inertial>
-      <mass value="1.0" />
-      <inertia ixx="1.0" ixy="0.0" ixz="0.0" iyy="1.0" iyz="0.0" izz="1.0"/>
+      <mass value="5.0" />
+      <!--<inertia ixx="${0.0833333 * scoop_mass * (scoop_width*scoop_width + (scoop_diameter/2)*(scoop_diameter/2))}" ixy="0.0" ixz="0.0"
+        iyy="${0.0833333 * scoop_mass * (scoop_length*scoop_length + (scoop_diameter/2)*(scoop_diameter/2))}" iyz="0.0"
+        izz="${0.0833333 * scoop_mass * (scoop_length*scoop_length + scoop_width*scoop_width)}" />-->
+      <inertia ixx="5.0" ixy="0.0" ixz="0.0" iyy="5.0" iyz="0.0" izz="5.0"/>
     </inertial>
   </link>
@@ -196,10 +226,10 @@
   <transmission name="scoop_tran">
     <type>transmission_interface/SimpleTransmission</type>
-    <joint name="end_to_arm">
-      <hardwareInterface>hardware_interface/EffortJointInterface
+    <joint name="scoop_joint">
+      <hardwareInterface>hardware_interface/PositionJointInterface
       </hardwareInterface>
     </joint>
     <actuator name="end_motor">
-      <hardwareInterface>hardware_interface/EffortJointInterface
+      <hardwareInterface>hardware_interface/PositionJointInterface
       </hardwareInterface>
       <mechanicalReduction>1</mechanicalReduction>
