Commit message: fix gazebo filse so that model of the arm does not destroy rviz simulation

File: src/tfr_description/xacro/model_constants.xacro (robot description, xacro)
@@ -16,4 +16,6 @@
   <xacro:property name="drivebase_total_height" value="${6*itom}" />
   <!-- Drivetrain parameters -->
+  <xacro:property name="tred_left_mass" value="${30.0}" />
+  <xacro:property name="tred_right_mass" value="${30.0}" />
   <xacro:property name="tread_end_radius" value="${(15.5/2)*itom}" />
   <xacro:property name="tread_mid_height" value="${19*itom}" />
@@ -26,4 +28,5 @@
   <!-- Length of top of bin, length of bottom is 13.86 -->
   <!-- Using the bigger size as a box instead of making complex angled shape -->
+  <xacro:property name="bin_mass" value="${10.0}" />
   <xacro:property name="bin_length" value="${36*itom}" />
   <xacro:property name="bin_width" value="${13.5*itom}" />
@@ -38,5 +41,5 @@
   <xacro:property name="turntable_height" value="${2.25*itom}" />
   <!-- Lower arm parameters -->
-  <xacro:property name="lower_arm_mass" value="${15.0}"/>
+  <xacro:property name="lower_arm_mass" value="${28.0}"/>
   <xacro:property name="lower_arm_length" value="${22*itom}" />
   <xacro:property name="lower_arm_primary_length" value="${16*itom}" />
